File: Uniformity Sensor.brd (EAGLE design)
At the start: 100 x 80 mm, 37 parts, among them IC1 SI1145, J3 USB-MICRO!!!, J4 3x2M, U1 ATMEGA32U4-XUMU, U4 LP2985-33DBVR, Y3 16MHz KX-7

Commit message: some routing
Parts:
- C5: device SmartPrj:C0402 -> arduino-micro-reference-designArduino_Micro_Rev03j:SMARTPRJ_C0603-ROUND
- moved D2 33.7 mm to (13.6, 1.65)
- moved R1 32.8 mm to (10.3, 1.65), turned to 90 degrees
- moved RX 26.7 mm to (9.78, 9.53), turned to 90 degrees
- moved C11 26.7 mm to (17.8, 1.27)
- moved C8 19.9 mm to (34.3, 12.7)
- moved R7 19.4 mm to (11.3, 11.6), turned to 180 degrees
- moved C10 18.3 mm to (26.7, 1.27)
- moved L 11.7 mm to (24.1, 15.2), turned to 0 degrees
- moved C12 9.35 mm to (16.6, 6.86), turned to 270 degrees
- moved C13 7.91 mm to (22.1, 6.60), turned to 90 degrees
- moved Y3 6.04 mm to (19.6, 6.60)
- moved R6 4.02 mm to (25.4, 5.08)
- moved Z2 2.84 mm to (8.89, 17.5), turned to 90 degrees
- moved F1 2.62 mm to (7.11, 22.1), turned to 0 degrees
- moved R8 2.54 mm to (22.9, 15.2), turned to 270 degrees
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Routing:
- net GND: track 0.00 -> 94.6 mm
- net VUSB: track 0.00 -> 56.5 mm
- net RESET: track 0.00 -> 24.4 mm
- net MOSI: track 0.00 -> 9.44 mm
- net VUSBD: track 0.00 -> 8.94 mm
- net SCK: track 0.00 -> 7.63 mm
- net D+: track 0.00 -> 6.03 mm
- net D-: track 0.00 -> 5.80 mm
- net MISO: track 0.00 -> 4.97 mm
- net RXLED/SS: track 0.00 -> 3.34 mm
- net AVCC: track 0.00 -> 2.85 mm
- net UCAP: track 0.00 -> 2.78 mm
- net RD-: track 0.00 -> 2.58 mm
- net RD+: track 0.00 -> 2.49 mm
- net N$2: track 0.00 -> 2.06 mm
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
Commit message: probably routed
Parts:
- removed RX, TX: yellow, led:CHIPLED_0805
- removed U$37: FIDUCIALMOUNT, SmartPrj:FIDUCIA-MOUNT
- removed U$53: FIDUCIAL1X2, SparkFun:FIDUCIAL-1X2
- added Q1, Q2: 200mA/50V, SparkFun-DiscreteSemi:SOT23-3
- added R3, R9: (no value), arduino-micro-reference-designArduino_Micro_Rev03j:SMARTPRJ_R0402
- J3: device SmartPrj:CON2_USB_MICRO_B_AT -> SparkFun-Connectors:USB-B-MICRO-SMD_V03
- R6: value 1K -> (none); device SmartPrj:R0402 -> arduino-micro-reference-designArduino_Micro_Rev03j:SMARTPRJ_R0402
- R7: value 1K -> (none); device SmartPrj:R0402 -> arduino-micro-reference-designArduino_Micro_Rev03j:SMARTPRJ_R0603-ROUND
- moved C11 23.7 mm to (24.1, 24.1), turned to 180 degrees
- moved R7 19.3 mm to (30.5, 14.0), turned to 90 degrees
- moved U4 16.6 mm to (27.9, 26.7)
- moved C10 15.2 mm to (26.7, 16.5), turned to 270 degrees
- moved C4 14.9 mm to (31.8, 26.7), turned to 270 degrees
- moved R6 10.5 mm to (35.6, 7.62), turned to 270 degrees
- moved ON 9.04 mm to (18.5, 30.9)
- moved R5 8.98 mm to (15.2, 30.5)
- moved L 8.83 mm to (30.9, 21.0), turned to 270 degrees
- moved C9 8.13 mm to (17.8, 27.9), turned to 270 degrees
- moved C6 7.41 mm to (20.3, 25.1)
- moved R2 7.41 mm to (15.2, 27.9), turned to 90 degrees
- moved R8 7.32 mm to (27.4, 21.0), turned to 0 degrees
- moved R4 7.18 mm to (27.9, 23.2)
- moved C7 6.84 mm to (17.8, 25.1)
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Connections:
- net 3V3: now also Q1.1, Q2.1, R3.2, R6.2
- net D+: now also J3.D+; no longer J3.P3
- net D-: now also J3.D-; no longer J3.P2
- net GND: now also J3.GND, J3.SHIELD1, J3.SHIELD2, J3.SHIELD3; no longer J3.P5, J3.S1, J3.S2, J3.S3, J3.S4, J3.S5, J3.S6, RX.C, TX.C
- net IO11*: no longer IC1.4
- net N$2: now also IC1.1, Q1.2, R3.1; no longer R7.2, RX.A
- net N$4: now also IC1.2, Q2.2, R6.1; no longer R6.2, TX.A
- net RXLED/SS: no longer R7.1
- net SCL: now also Q2.3, R7.1; no longer IC1.2
- net SDA: now also Q1.3, R9.1; no longer IC1.1
- net TXLED: no longer R6.1
- net VUSB: now also R7.2, R9.2
- net VUSBD: now also J3.VBUS; no longer J3.P1
Routing:
- net VUSB: track 56.5 -> 95.1 mm, vias 0 -> 3
- net 3V3: track 0.00 -> 38.5 mm
- net GND: track 94.6 -> 114.9 mm, vias 0 -> 16
- net SCL: track 0.00 -> 13.8 mm
- net SDA: track 0.00 -> 12.4 mm
- net XTAL2: track 0.00 -> 8.26 mm
- net XTAL1: track 0.00 -> 7.85 mm
- net N$4: track 0.00 -> 7.74 mm
- net N$2: track 2.06 -> 6.17 mm
- net RESET: track 24.4 -> 28.2 mm
- net VUSBD: track 8.94 -> 12.6 mm
- net HWB: track 0.00 -> 3.59 mm
- net RXLED/SS: track 3.34 -> 0.00 mm
- net AVCC: track 2.85 -> 5.66 mm
- net RD+: track 2.49 -> 5.03 mm
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- added copper zone on layer 16, net GND
- added copper zone on layer 1, net N$5
- added copper zone on layer 1, net VUSB
Other:
- board size 100 x 80 mm -> 43.2 x 34.3 mm

Commit message: Gerber and BOM
Routing:
- net VUSB: track 95.1 -> 88.2 mm, vias 3 -> 2
Changed lines of the file:
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@@
 <wire x1="16.585" y1="21.05" x2="18.315" y2="21.05" width="0.3048" layer="1"/>
 <wire x1="18.315" y1="18.55" x2="16.01" y2="18.55" width="0.3048" layer="1"/>
-<wire x1="16.01" y1="18.55" x2="15.24" y2="17.78" width="0.3048" layer="1"/>
-<wire x1="15.24" y1="17.78" x2="13.97" y2="16.51" width="0.3048" layer="1"/>
+<wire x1="16.01" y1="18.55" x2="13.97" y2="16.51" width="0.3048" layer="1"/>
 <wire x1="13.97" y1="16.51" x2="13.335" y2="16.51" width="0.3048" layer="1"/>
 <wire x1="13.335" y1="16.51" x2="12.7" y2="17.145" width="0.3048" layer="1"/>
@@
 <via x="20.066" y="12.954" extent="1-16" drill="0.6" shape="octagon"/>
 <wire x1="20.066" y1="12.954" x2="20.066" y2="13.081" width="0.3048" layer="16"/>
-<wire x1="20.066" y1="13.081" x2="15.3035" y2="17.8435" width="0.3048" layer="16"/>
-<via x="15.24" y="17.78" extent="1-16" drill="0.6" shape="octagon"/>
 <wire x1="24.865" y1="17.05" x2="26.67" y2="17.05" width="0.3048" layer="1"/>
 <wire x1="26.67" y1="17.05" x2="26.67" y2="18.161" width="0.3048" layer="1"/>
@@
 <wire x1="26.67" y1="18.161" x2="25.273" y2="18.161" width="0.3048" layer="16"/>
 <wire x1="25.273" y1="18.161" x2="20.066" y2="12.954" width="0.3048" layer="16"/>
-<wire x1="15.3035" y1="17.8435" x2="15.24" y2="17.78" width="0.3048" layer="16"/>
 <polygon width="0.3048" layer="1" spacing="0.4064" isolate="0.3048">
 <vertex x="0" y="34.29"/>
